File: AL_Controller.sch (KiCad schematic (older format))
At the start: 5 parts

Commit message: misc updatees
Parts:
- gave numbers to parts that had none: 5
Changed lines of the file:
@@
 Ins3
 $Comp
-L CPU_internal_elements:OctalBuffer U?
+L CPU_internal_elements:OctalBuffer U25
 U 1 1 610132D8
 P 3050 1300
-F 0 "U?" H 3050 1275 50  0000 C CNN
+F 0 "U25" H 3050 1275 50  0000 C CNN
 F 1 "OctalBuffer" H 3050 1184 50  0000 C CNN
 F 2 "" H 3050 1300 50  0001 C CNN
@@
 	2300 2250 2750 2250
 $Comp
-L 74xGxx:74AHC1G08 U?
+L 74xGxx:74AHC1G08 U23
 U 1 1 6101A286
 P 2750 2650
-F 0 "U?" V 2725 2520 50  0000 R CNN
+F 0 "U23" V 2725 2520 50  0000 R CNN
 F 1 "74AHC1G08" H 2725 2826 50  0001 C CNN
 F 2 "" H 2750 2650 50  0001 C CNN
@@
 	2300 3300 2600 3300
 $Comp
-L 74xGxx:74AHC1G08 U?
+L 74xGxx:74AHC1G08 U24
 U 1 1 61022A3F
 P 2900 3250
-F 0 "U?" H 3050 3150 50  0000 C CNN
+F 0 "U24" H 3050 3150 50  0000 C CNN
 F 1 "a" H 2950 3000 50  0001 C CNN
 F 2 "" H 2900 3250 50  0001 C CNN
@@
 B3
 $Comp
-L CPU_internal_elements:74181 U?
+L CPU_internal_elements:74181 U21
 U 1 1 61026E63
 P 1250 700
-F 0 "U?" H 1525 725 50  0000 C CNN
+F 0 "U21" H 1525 725 50  0000 C CNN
 F 1 "74181" H 1525 634 50  0000 C CNN
 F 2 "" H 1250 700 50  0001 C CNN
@@
 $EndComp
 $Comp
-L CPU_internal_elements:74181 U?
+L CPU_internal_elements:74181 U22
 U 1 1 61029705
 P 1300 2250
-F 0 "U?" H 1575 2275 50  0000 C CNN
+F 0 "U22" H 1575 2275 50  0000 C CNN
 F 1 "74181" H 1575 2184 50  0000 C CNN
 F 2 "" H 1300 2250 50  0001 C CNN
