File: MAX7000CPU.sch (KiCad schematic (older format))
At the start: 118 parts, among them J1 Conn_02x05_Odd_Even, J2 Conn_01x08_Male, J3 Conn_01x08_Male, J4 Conn_01x08_Male, J5 Conn_01x08_Male, J6 Conn_01x08_Male, J7 Conn_01x05_Male, J8 Barrel_Jack, SW1 SW_Push, SW2 SW_Push, SW3 SW_DIP_x04, SW4 SW_Push, U1 NE555P, U10 74LS573, U11 74LS241, U12 74LS241, U13 74LS573, U14 74LS573, U15 74LS573, U16 74LS573, U17 EPM7128slc84-15n, U18 LM2596S-5, U19 74LS241, U2 NE555P, U20 74LS241, U3 NE555P, U4 CLVC1GX04MDRLREP, U5 EPM7128slc84-15n, U6 74LS573, U7 SN74HC161N, U8 SN74HC161N, U9 IDT7132, Y1 Crystal

Commit message: misc updatees
Connections:
- no-connect marks 18 -> 19
Other:
- note added: "CRITICAL FLAW: THESE REGISTERS NEED TO BE TIED LOW NOT HIGH"
Changed lines of the file:
@@
 Text Label 2500 5350 0    50   ~ 0
 O3
+$Sheet
+S 3250 5050 900  600
+U 60FFC927
+F0 "U5 ALC Architechture" 50
+F1 "AL_Controller.sch" 50
+$EndSheet
+NoConn ~ 3100 5500
+Text Notes 11500 600  0    50   ~ 0
+CRITICAL FLAW: THESE REGISTERS NEED TO BE TIED LOW NOT HIGH
 Wire Bus Line
 	8800 4150 8800 4350
@@
 Wire Bus Line
 	4600 7900 4600 8800
-$Sheet
-S 3250 5050 900  600
-U 60FFC927
-F0 "U5 ALC Architechture" 50
-F1 "AL_Controller.sch" 50
-$EndSheet
 $EndSCHEMATC
